File: Cap_Water_Sensor_Eagle/GWLSensorv5.brd (EAGLE design)
At the start: 13 parts, among them IC1 LM555D

Commit message: V6
Parts:
- moved C1 33.4 mm to (8.89, 41.5)
- moved C2 33.4 mm to (7.62, 32.6)
- moved C3 33.4 mm to (10.2, 19.9)
- moved D1 33.4 mm to (20.3, 42.8)
- moved SIGNAL 33.4 mm to (48.8, 48.6)
- moved C4 33.4 mm to (30.5, 49.1)
- moved IC1 33.4 mm to (24.1, 28.8)
- moved R1 33.4 mm to (34.3, 30.1)
- moved R2 33.4 mm to (16.5, 50.4)
- moved R3 33.4 mm to (38.1, 49.1)
- moved RA 33.4 mm to (40.6, 30.1)
- moved SENSOR 33.4 mm to (9.02, 57.7)
- moved VCC/GND 33.4 mm to (10.2, 8.26)
Routing:
- net N$4: track 10.6 -> 0.00 mm
- net N$7: track 3.23 -> 0.00 mm
