File: Cap_Water_Sensor_Eagle/GWLSensorv6.brd (EAGLE design)
At the start: 13 parts, among them IC1 LM555D

Commit message: V6
Parts:
- D1: value 1N4004 -> (none); device diode:DO41-10 -> adafruit:SMADIODE
- moved SENSOR 44.0 mm to (-13.2, 53.0), turned to 270 degrees
- moved C1 36.6 mm to (15.1, 38.9), turned to 270 degrees
- moved R2 35.4 mm to (-1.26, 53.2), turned to 270 degrees
- moved RA 34.4 mm to (9.60, 48.7), turned to 90 degrees
- moved SIGNAL 34.2 mm to (30.6, 53.1)
- moved R3 34.2 mm to (20.8, 53.1), turned to 270 degrees
- moved C4 33.2 mm to (15.1, 53.1), turned to 270 degrees
- moved R1 32.5 mm to (5.26, 48.8), turned to 270 degrees
- moved IC1 29.0 mm to (5.71, 39.8)
- moved C2 26.2 mm to (11.5, 40.1), turned to 90 degrees
- moved D1 25.7 mm to (7.33, 54.1)
- moved VCC/GND 23.4 mm to (-13.2, 40.6), turned to 270 degrees
- moved C3 19.0 mm to (-3.96, 40.7), turned to 90 degrees
Routing:
- net VCC: track 0.00 -> 92.5 mm, vias 0 -> 1
- net GND: track 0.00 -> 83.0 mm
- net N$7: track 3.23 -> 37.4 mm, vias 0 -> 2
- net N$6: track 0.00 -> 20.0 mm
- net N$1: track 0.00 -> 19.2 mm
- net N$4: track 10.6 -> 29.4 mm, vias 0 -> 1
- net N$3: track 0.00 -> 16.2 mm
- net N$2: track 0.00 -> 15.4 mm
