File: Cap_Water_Sensor_Eagle/GWLSensorv6.brd (EAGLE design)
At the start: 13 parts, among them IC1 LM555D

Commit message: v6 with no blue lines
Routing:
- net VCC: track 92.5 -> 47.0 mm
- net N$7: track 37.4 -> 17.3 mm
- net N$4: track 29.4 -> 10.6 mm
Changed lines of the file:
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@@
 <contactref element="IC1" pad="5"/>
 <contactref element="C1" pad="2"/>
-<wire x1="24.384" y1="26.9748" x2="16.9164" y2="34.4424" width="0.1524" layer="16"/>
-<wire x1="16.9164" y1="34.4424" x2="17.6784" y2="35.2044" width="0.1524" layer="16"/>
-<wire x1="17.6784" y1="35.2044" x2="22.7076" y2="40.2336" width="0.1524" layer="16"/>
 <wire x1="8.382" y1="37.9476" x2="15.0876" y2="37.9476" width="0.1524" layer="1"/>
 <wire x1="15.0876" y1="37.9476" x2="15.0876" y2="37.912" width="0.1524" layer="1"/>
@@
 <contactref element="IC1" pad="3"/>
 <contactref element="R2" pad="2"/>
-<wire x1="19.9644" y1="28.8036" x2="19.9644" y2="28.956" width="0.1524" layer="16"/>
-<wire x1="19.9644" y1="28.956" x2="7.3152" y2="41.6052" width="0.1524" layer="16"/>
 <wire x1="-1.2192" y1="50.1396" x2="-1.2192" y2="52.1208" width="0.1524" layer="1"/>
-<wire x1="7.3152" y1="41.6052" x2="-1.2192" y2="50.1396" width="0.1524" layer="16"/>
 <wire x1="-1.2192" y1="52.1208" x2="-1.2576875" y2="52.209946875" width="0.1524" layer="1"/>
 <wire x1="4.8768" y1="39.1668" x2="3.115" y2="39.1668" width="0.1524" layer="1"/>
-<wire x1="7.3152" y1="41.6052" x2="4.8768" y2="39.1668" width="0.1524" layer="16"/>
 <via x="-1.2192" y="50.1396" extent="1-16" drill="0.35"/>
 <via x="4.8768" y="39.1668" extent="1-16" drill="0.35"/>
+<wire x1="-1.2192" y1="45.2628" x2="-1.2192" y2="50.1396" width="0.1524" layer="16"/>
+<wire x1="4.8768" y1="39.1668" x2="-1.2192" y2="45.2628" width="0.1524" layer="16"/>
 </signal>
 <signal name="VCC">
@@
 <contactref element="IC1" pad="4"/>
 <contactref element="RA" pad="1"/>
-<wire x1="24.9936" y1="29.718" x2="24.0792" y2="28.8036" width="0.1524" layer="16"/>
-<wire x1="24.6888" y1="26.8224" x2="24.384" y2="26.5176" width="0.1524" layer="16"/>
-<wire x1="24.384" y1="26.5176" x2="17.8308" y2="19.9644" width="0.1524" layer="16"/>
-<wire x1="24.6888" y1="28.194" x2="24.6888" y2="26.8224" width="0.1524" layer="16"/>
-<wire x1="24.0792" y1="28.8036" x2="24.6888" y2="28.194" width="0.1524" layer="16"/>
-<wire x1="35.9664" y1="29.718" x2="24.9936" y2="29.718" width="0.1524" layer="16"/>
 <wire x1="9.6012" y1="42.9768" x2="9.6012" y2="47.7672" width="0.1524" layer="1"/>
 <wire x1="8.382" y1="41.7576" x2="9.2964" y2="42.672" width="0.1524" layer="1"/>
@@
 <wire x1="9.6012" y1="47.8536" x2="9.6012" y2="47.7672" width="0.1524" layer="1"/>
 <wire x1="-3.9624" y1="41.7576" x2="-3.9624" y2="41.6408" width="0.1524" layer="1"/>
-<wire x1="9.2964" y1="41.6052" x2="24.384" y2="26.5176" width="0.1524" layer="16"/>
 <wire x1="9.2964" y1="42.672" x2="9.2964" y2="41.6052" width="0.1524" layer="16"/>
 <via x="9.2964" y="42.672" extent="1-16" drill="0.35"/>
