File: Cap_Water_Sensor_Eagle/FD Capacitance Sensor v06.brd (EAGLE design)
At the start: 160 x 100 mm, 17 parts, among them U1 NTS4101PT1, U2 TLC555CD

Commit message: More updates
Parts:
- moved J1 30.3 mm to (3.10, 5.38), turned to 0 degrees
- moved D2 11.5 mm to (17.0, 10.7)
- moved C8 8.82 mm to (24.9, 16.0), turned to 180 degrees
- moved OUTPUT 6.40 mm to (27.7, 4.62)
- moved C9 3.02 mm to (8.41, 20.2), turned to 90 degrees
- moved C10 1.86 mm to (17.1, 12.8)
- moved R6 1.78 mm to (6.10, 20.3), turned to 270 degrees
- moved R9 0.69 mm to (20.8, 12.9)
- moved R5 0.65 mm to (11.9, 17.2)
- moved C2 0.13 mm to (23.6, 22.4)
Routing:
- net OUTPUT1: track 28.0 -> 15.3 mm
- net N$9: track 36.6 -> 25.0 mm, vias 2 -> 0
- net SENSOR1: track 11.9 -> 20.7 mm
- net +3V3: track 11.0 -> 17.6 mm
- net !EN: track 8.26 -> 14.8 mm
- net N$8: track 25.1 -> 27.7 mm, vias 2 -> 0
- net N$1: track 4.75 -> 3.79 mm, vias 2 -> 0
- net N$5: track 3.22 -> 2.58 mm
- net VCC: vias 0 -> 1

Commit message: Newest BRD
Parts:
- removed FRAME1: FRAME-LETTERNO_PACKAGE, SparkFun-Aesthetics:DUMMY
- moved D2 0.74 mm to (17.6, 11.2)
- moved U1 0.74 mm to (24.2, 20.1)
- moved C6 0.74 mm to (6.81, 16.3)
- moved C7 0.74 mm to (6.81, 12.3)
- moved R6 0.74 mm to (6.68, 20.8)
- moved R8 0.74 mm to (8.38, 14.2)
- moved C10 0.74 mm to (17.7, 13.3)
- moved C8 0.74 mm to (25.5, 16.5)
- moved C9 0.74 mm to (8.99, 20.7)
- moved OUTPUT 0.74 mm to (28.3, 5.08)
- moved R5 0.74 mm to (12.4, 17.7)
- moved R7 0.74 mm to (27.4, 20.2)
- moved R9 0.74 mm to (21.4, 13.3)
- moved U2 0.74 mm to (18.4, 18.2)
- moved J1 0.74 mm to (3.68, 5.84)
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Other:
- board size 160 x 100 mm -> 35.1 x 27.6 mm
