File: Cap_Water_Sensor_Eagle/FD Capacitance Sensor v11.brd (EAGLE design)
At the start: 38.6 x 34 mm, 21 parts, among them J1 BM06B-SRSS-TBT(LF)(SN), U1 NTS4101PT1, U2 TLC555CD

Commit message: v11
Parts:
- moved C4 16.5 mm to (20.7, 9.54)
- moved C5 6.67 mm to (15.8, 9.44), turned to 0 degrees
- moved R1 0.25 mm to (15.5, 24.6)
Routing:
- net N$1: track 21.6 -> 2.16 mm
- net N$5: track 10.4 -> 13.6 mm
- net N$8: track 22.1 -> 19.2 mm
- net OUTPUT1: track 12.5 -> 14.4 mm
- net VCC: track 41.3 -> 39.5 mm
- net SENSOR1: track 23.0 -> 22.1 mm
- net !EN: track 11.9 -> 12.6 mm
